File: 700CDockSlotFlipped.kicad_pcb (KiCad board)
At the start: 2 copper layers, 94 x 77 mm, 21 parts, among them J1 BUS_MCA, J10 GND, J100 Conn_02x60, J2 UPPER, J3 HPLA_PORT, J4 HPLA_PORT, J5 HPLA_PORT, J6 HPLA_PORT, J7 IRQ, J8 5V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

Commit message: Rev 2: Fix CHRESET, disconnect and pull up MADE24
Parts:
- removed U3: MAX810LTRG, Active:SOT95P230X117-3
- moved R3 56.7 mm to (100.3, 79.8), turned to -90 degrees
Connections:
- J100 pad 102: /MADE24 -> /CHRST
- R3 pad 1: /CHRST -> +5C
- R3 pad 2: GND -> /MADE24
Routing:
- net /MADE24: track 196.8 -> 113.0 mm, vias 6 -> 4
- net /CHRST: track 29.5 -> 45.4 mm
- net +5C: track 204.0 -> 202.3 mm, vias 5 -> 6
- net /~{CD_SETUP}: track 100.5 -> 101.0 mm
- net GND: vias 71 -> 75
